File: PowerConverter.kicad_sch (KiCad schematic)
At the start: 9 parts, among them U4 XL1509-5.0E1, U5 AMS1117-3.3

Commit message: Done routing for Buck Converter , Rs485 and CAN , Some Routing for MCU and associated circuitry , NO ETHERNET ROUTING , NO module Interconnects yet
Parts:
- C18: footprint Capacitor_THT:CP_Radial_D6.3mm_P2.50mm -> Capacitor_THT:CP_Radial_D8.0mm_P3.50mm
Changed lines of the file:
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@@
 			)
 		)
-		(property "Footprint" "Capacitor_THT:CP_Radial_D6.3mm_P2.50mm"
+		(property "Footprint" "Capacitor_THT:CP_Radial_D8.0mm_P3.50mm"
 			(at 113.9952 88.9 0)
 			(effects
