File: Esp32.kicad_sch (KiCad schematic)
At the start: 11 parts, among them J2 Conn_01x03_Pin, J3 Conn_01x02_Pin, J4 Conn_01x05_Pin, SW4 SW_Push, U6 AMS1117-3.3, U7 ESP32-WROOM-32

Commit message: UPDATED
Parts:
- removed J4: Conn_01x05_Pin, symbol Connector:Conn_01x05_Pin
- added D1, D2, D5: LED, LED_SMD:LED_1206_3216Metric_Pad1.42x1.75mm_HandSolder, symbol Device:LED
- added J4: Conn_01x03_Pin, Connector_PinHeader_2.54mm:PinHeader_1x03_P2.54mm_Horizontal, symbol Connector:Conn_01x03_Pin
- added R3, R4, R5: 1k, Resistor_SMD:R_1206_3216Metric_Pad1.30x1.75mm_HandSolder, symbol Device:R
- C3: footprint (none) -> Capacitor_SMD:C_1206_3216Metric_Pad1.33x1.80mm_HandSolder
- J2: footprint Connector_PinHeader_2.54mm:PinHeader_1x03_P2.54mm_Vertical -> Connector_PinHeader_2.54mm:PinHeader_1x03_P2.54mm_Horizontal
- J3: footprint Connector_PinHeader_2.54mm:PinHeader_1x02_P2.54mm_Vertical -> Connector_PinHeader_2.54mm:PinHeader_1x02_P2.54mm_Horizontal
- R1, R2: footprint (none) -> Resistor_SMD:R_1206_3216Metric_Pad1.30x1.75mm_HandSolder
Connections:
- net +3.3VESP: now also R3.1, R4.1, R5.1
- net GND: now also J3.2 (Pin_2), J4.3 (Pin_3); no longer J3.1 (Pin_1)
- net at U7.25 (IO0): now also J3.1 (Pin_1); no longer J3.2 (Pin_2)
- net INDESP_LED0: now reaches U7.10 (IO25)
- net INDESP_LED0: now also D5.1 (K)
- net INDESP_LED1: now reaches U7.11 (IO26)
- net INDESP_LED1: now also D1.1 (K)
- net INDESP_LED2: now reaches U7.12 (IO27)
- net INDESP_LED2: now also D2.1 (K)
- net SPI_CLK: now reaches U7.13 (IO14)
- net SPI_MISO: now reaches U7.14 (IO12)
- net SPI_MOSI: now reaches U7.16 (IO13)
- net SPI_CS: now reaches U7.23 (IO15)
- net at U7.27 (IO16): now also J4.2 (Pin_2)
- net at U7.28 (IO17): now also J4.1 (Pin_1)
- net at U7.34 (RXD0): now also J2.1 (Pin_1); no longer J2.2 (Pin_2)
- net at U7.35 (TXD0): now also J2.2 (Pin_2); no longer J2.1 (Pin_1)
- new net: D5.2 (A), R5.2
- new net: D1.2 (A), R4.2
- new net: D2.2 (A), R3.2
Other:
- moved on the sheet: C3, J3, R1, R2, SW4

Commit message: Latest Changes
Parts:
- SW4: footprint (none) -> Button_Switch_SMD:SW_SPST_CK_RS282G05A3
Changed lines of the file:
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@@
 			)
 		)
-		(property "Footprint" ""
+		(property "Footprint" "Button_Switch_SMD:SW_SPST_CK_RS282G05A3"
 			(at 69.85 62.23 0)
 			(effects
